File: hardware/v2_board/board.sch (EAGLE design)
At the start: 144 parts, among them IC1 AVR_XMEGA_A3_, Q1 RESONATORSMD, U1 ATMEGA168, U16 BSS138AKA, U2 STM32F415RGT6, U6 BSS138AKA, X1 MINI-USB-UX60A-MB-5ST

Commit message: + Osazovací výkresy
Parts:
- C14, C15, C16, C17, C18, C20, C21, C29, C30: value 0.1uF -> 100nF
- LED10, LED12, LED8: value RED -> YELLOW
- LED11, LED13, LED9: value GREEN -> YELLOW
- LED14: value (none) -> BLUE
- LED15: value (none) -> YELLOW
- Q1: value RESONATORSMD -> 16MHz
- R10, R11, R12, R5, R6, R7, R8, R9: value 10k -> 1k
- R2, R21, R26, R27, R30, R31, R32, R33, R34, R35, R40, R41: value 330R -> 470R
- R22, R28: value 330R -> 1k
- R23, R24, R25: value 330R -> 120R
- R29, R42: value 330R -> 270R
- RSSI: value BLUE -> YELLOW

Commit message: + scheme polished & schema png
Other:
- note added: "Blocking capacitors"
- note added: "LEDs"
- note added: "Micro-controllers"
- note added: "Power supply input part"
- note added: "Programming connectors & USB"
- note added: "xBee wireless module"
- note added: "xMega I/O"
- note removed: "OBC"
- note removed: "Serial I/O"
- note removed: "Switching power supply"
- note removed: "Test points"
- note removed: "Wireless module"
- moved on the sheet: C10, C11, C12, C13, C14, C15, C16, C17, C19, C20, C21, C22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
